Commit message: updated files

File: IsaacSim Models/Test_Bench_Model/test_bench with joint specs.urdf (robot description, URDF)
Before this commit: robot test_bench, 4 links, 3 joints
Joints:
- joint revolute_lift: limit lower=0.1745329252 upper=1.6057029118 effort=0 velocity=0 -> lower=0.1745329252 upper=1.6057029118 effort=60 velocity=0.5
- joint revolute_scoop: limit lower=-0.5235987756 upper=1.1344640138 effort=0 velocity=0 -> lower=-0.5235987756 upper=1.1344640138 effort=30 velocity=0.5
- joint revolute_tilt: limit lower=-0.4886921906 upper=1.4835298642 effort=0 velocity=0 -> lower=-0.4886921906 upper=1.4835298642 effort=30 velocity=0.5
