Commit message: Updated urdf file

File: IsaacSim Models/Excavator_Model/Excavator_v1.urdf (robot description, URDF)
Before this commit: robot Excavator, 5 links, 4 joints
Links:
- link liftboom: geometry collision mesh filename=.\Assets\liftboom.stl; visual mesh filename=.\Assets\liftboom.stl
- link scoop: geometry collision mesh filename=.\Assets\scoopandmount.stl; visual mesh filename=.\Assets\scoopandmount.stl
- link tiltboom: geometry collision mesh filename=.\Assets\tiltboom.stl; visual mesh filename=.\Assets\tiltboom.stl
- link uppercarriage: geometry collision mesh filename=.\Assets\uppercarriage.stl; visual mesh filename=.\Assets\uppercarriage.stl
